File: hardware/tspico-v3.kicad_sch (KiCad schematic)
At the start: 0 parts

Commit message: Emulated memory: rewrite architecture, add local-bus/register sheet
- docs/v3-architecture.md: RP2350B serves DCK/ROM images from internal SRAM
  via PIO+DMA; no flash or SRAM chips; 8-bit multiplexed local bus; slot map
  file replaces fixed flash banks; ESP32-C3-WROOM-02 for Zimodem.
- memory sheet: 74LVC257 address byte muxes, ALO/AHI/CTL/STAT registers,
  74LVC139 select, power-on clear for CTL.
- interface sheet: 74LVC06 inverting open-drain drivers with active-high
  requests (safe power-up state), RESET_HOLD pull-up, address transceivers
  always enabled, MA8-MA15 to the muxes, WIFI_DL inverter.
- ERC: only cross-sheet labels/inputs pending the MCU and peripheral sheets.

Co-Authored-By: Claude Fable 5.1 <noreply@anthropic.com>
Other:
- sheet Memory Bus renamed Local Bus and Registers
Changed lines of the file:
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@@
   )
   (sheet (at 110.0 30.0) (size 60 30) (fields_autoplaced yes) (stroke (width 0.1524) (type solid)) (fill (color 0 0 0 0.0000))
-    (property "Sheetname" "Memory Bus" (at 110.0 29.3 0) (effects (font (size 1.27 1.27)) (justify left bottom)))
+    (property "Sheetname" "Local Bus and Registers" (at 110.0 29.3 0) (effects (font (size 1.27 1.27)) (justify left bottom)))
     (property "Sheetfile" "memory.kicad_sch" (at 110.0 60.6 0) (effects (font (size 1.27 1.27)) (justify left top)))
     (instances (project "tspico-v3" (path "/9088d141-8624-4d5c-91a9-7a3a7a90b3cc" (page "3"))))
