File: hardware/wifi.kicad_sch (KiCad schematic)
At the start: 4 parts, among them U40 ESP32-C3-WROOM-02-N4

Commit message: Logic consolidation: 15 packages to 8 fitted
Address buffers' output enables replace the 74LVC257 byte muxes and the MA bus;
one 74LVC32 makes MEMRD/MEMWR/IORD/IOWR strobes (replaces the 04 and 08);
XL9555 I2C expander replaces the CTL register, its power-on clear and the STAT
buffer; DMA parts are a DNP stuffing option (config.DMA_OPTION), with 74LVC574
latches directly on the address bus. GPIO map, architecture doc and cost notes
updated. Parts + fees per board now $14.93 on a 10-board run.

Co-Authored-By: Claude Fable 5.1 <noreply@anthropic.com>
Parts:
- added R41: 10k, Resistor_SMD:R_0603_1608Metric, symbol Device:R
Connections:
- net +3V3_WIFI: now also R41.1
- net nWIFI_BOOT: now also R41.2
Other:
- note added: "R40: IO8 must be high during a download-mode boot. IO9 low = download mode: R41 pulls it up, the open-drain gate in U7 pulls it down when WIFI_DL is set."
- note removed: "R40: IO8 must be high during a download-mode boot. IO9 low = download mode (driven by nWIFI_BOOT)."
Changed lines of the file:
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@@
   (global_label "+3V3_WIFI" (shape input) (at 229.87 86.36 90) (effects (font (size 1.27 1.27)) (justify left)))
   (label "ESP_IO8" (at 229.87 93.98 270) (effects (font (size 1.27 1.27)) (justify right bottom)))
+  (symbol (lib_id "Device:R") (at 245.11 90.17 0) (unit 1)
+    (exclude_from_sim no) (in_bom yes) (on_board yes) (dnp no)
+    (property "Reference" "R41" (at 248.11 81.86 0) (effects (font (size 1.27 1.27)) (justify left)))
+    (property "Value" "10k" (at 248.11 84.36 0) (effects (font (size 1.27 1.27)) (justify left)))
+    (property "Footprint" "Resistor_SMD:R_0603_1608Metric" (at 245.11 90.17 0) (effects (font (size 1.27 1.27)) (justify left) (hide yes)))
+    (property "Datasheet" "" (at 245.11 90.17 0) (effects (font (size 1.27 1.27)) (justify left) (hide yes)))
+    (property "Description" "" (at 245.11 90.17 0) (effects (font (size 1.27 1.27)) (justify left) (hide yes)))
+    (property "MPN" "0603WAF1002T5E" (at 245.11 90.17 0) (effects (font (size 1.27 1.27)) (justify left) (hide yes)))
+    (property "LCSC" "C25804" (at 245.11 90.17 0) (effects (font (size 1.27 1.27)) (justify left) (hide yes)))
+    (pin "1")
+    (pin "2")
+    (instances (project "tspico-v3" (path "/9088d141-8624-4d5c-91a9-7a3a7a90b3cc/d28d46ae-5d37-4c4f-b909-43ed531db596" (reference "R41") (unit 1))))
+  )
+  (global_label "+3V3_WIFI" (shape input) (at 245.11 86.36 90) (effects (font (size 1.27 1.27)) (justify left)))
+  (global_label "nWIFI_BOOT" (shape input) (at 245.11 93.98 270) (effects (font (size 1.27 1.27)) (justify right)))
   (symbol (lib_id "Device:C") (at 229.87 129.54 0) (unit 1)
     (exclude_from_sim no) (in_bom yes) (on_board yes) (dnp no)
@@
   (global_label "+3V3_WIFI" (shape input) (at 245.11 125.73 90) (effects (font (size 1.27 1.27)) (justify left)))
   (label "GND" (at 245.11 133.35 270) (effects (font (size 1.27 1.27)) (justify right bottom)))
-  (text "R40: IO8 must be high during a download-mode boot. IO9 low = download mode (driven by nWIFI_BOOT)." (exclude_from_sim no) (at 130 180 0) (effects (font (size 1.5 1.5)) (justify left bottom)))
+  (text "R40: IO8 must be high during a download-mode boot. IO9 low = download mode: R41 pulls it up, the open-drain gate in U7 pulls it down when WIFI_DL is set." (exclude_from_sim no) (at 130 180 0) (effects (font (size 1.5 1.5)) (justify left bottom)))
   (text "Zimodem's modem-status pins (DCD, RI, DSR, DTR, RTS/CTS) are not routed; XON/XOFF flow control." (exclude_from_sim no) (at 130 183 0) (effects (font (size 1.5 1.5)) (justify left bottom)))
   (embedded_fonts no)
