File: hardware-v2.6/logic.kicad_sch (KiCad schematic)
At the start: 20 parts, among them U1 74LS04, U4 74LS32, U5 74LS27, U6 74LVC245APW, U7 74LVC245APW, U8 74LS157, U9 74LS09

Commit message: v2.6 prototype 2: glue logic in 74LVC, TPS3808 reset
The v2.2 glue (74LS04/27/32/09/157) is rebuilt in 74LVC at 3.3 V, because
the SN74LS09 (56) and XL74LS27 (108) were scarce at JLCPCB and every glue
output already ends at a 3.3 V part. Same logic at every Pico pin, so no
firmware change:

- U5 74LVC138 decodes the port (A4-A6 select; /IORQ, A7, /M1 enables);
  JP4 now picks output O0 ($00-$0F) or O1 ($10-$1F)
- U4 74LVC32: /+RW (buffered so it keeps step with /+W), /+W = /+RW-select
  OR /RD, /RDROM = A14 + A15 + /RD
- U1 74LVC1G97 (mux wired as OR with one inverted input): /MREQ_G
- U9 74LVC2G07 open-drain /BE driver; U7 channel 5 now carries /BE_IN as
  /BE_STAT, so R4 and R7 go
- U8 74LVC157 for the A14/A15 mux
- U11 TPS3808G01 replaces the 555, Q1 and passives: /RESET held below
  4.09 V and for 2.7 s after (CT 470 nF)

Checked by simulating the old and new netlists gate by gate over all
229,376 legal input states, both JP4 positions: all 12 outputs agree. The
only difference is /+W when /M1, /IORQ and /RD are all low, which a Z80
never does.

Layout: the RP2040's top/bottom-row IOVDD caps stand on their own pin's
lane with locked pin-to-cap stubs; without that the router left one net
open on three attempts. Routed first time, ERC/DRC clean at every
severity. 74 assembled parts (was 81), $9.79/board at 10.

Co-Authored-By: Claude Opus 5.5 <noreply@anthropic.com>
Parts:
- removed R2, R7: 4k7, Resistor_SMD:R_0603_1608Metric, symbol Device:R
- removed U1: 74LS04, Package_SO:SOIC-14_3.9x8.7mm_P1.27mm, symbol 74xx:74LS04
- removed U5: 74LS27, Package_SO:SOIC-14_3.9x8.7mm_P1.27mm, symbol 74xx:74LS27
- removed U9: 74LS09, Package_SO:SOIC-14_3.9x8.7mm_P1.27mm, symbol 74xx:74LS09
- added U1: 74LVC1G97, Package_TO_SOT_SMD:SOT-23-6, symbol 74xGxx:74LVC1G97
- added U5: 74LVC138A, Package_SO:TSSOP-16_4.4x5mm_P0.65mm, symbol 74xx:74LS138
- added U9: 74LVC2G07, Package_TO_SOT_SMD:SOT-23-6, symbol 74xGxx:74LVC2G07
- U4: value 74LS32 -> 74LVC32A; footprint Package_SO:SOIC-14_3.9x8.7mm_P1.27mm -> Package_SO:TSSOP-14_4.4x5mm_P0.65mm; LCSC C116812 -> C6087; MPN SN74LS32DR -> 74LVC32APW,118
- U8: value 74LS157 -> 74LVC157A; footprint Package_SO:SOIC-16_3.9x9.9mm_P1.27mm -> Package_SO:TSSOP-16_4.4x5mm_P0.65mm; LCSC C707097 -> C406871; MPN XL74LS157 -> SN74LVC157APWR
Connections:
- net BE_IN is gone; now on net nRD: U4.13
- net BE_L_BUF is gone; now on net nBE_STAT: U7.14 (B4)
- net OR567 is gone; now on net A14: U4.9
- net PX is gone; now on net A14_OR_A15: U4.8
- net U7_DIR is gone; now on net +3V3: U7.1 (A->B)
- net +3V3: now also C1.1, C14.1, C4.1, C5.1, C8.1, U4.14 (VCC), U8.16 (VCC), U1.1 (IN1), U1.5 (VCC), U5.16 (VCC), U9.5 (VCC)
- net +5V: no longer C1.1, C14.1, C4.1, C5.1, C8.1, U4.14 (VCC), U8.16 (VCC)
- net A14: no longer U4.1
- net A14_OR_A15: now also U4.12; no longer U4.3, U4.4
- net A15: now also U4.10; no longer U4.2
- net A4: now also U5.1 (A0); no longer JP4.1 (A)
- net A5: now also U5.2 (A1)
- net A6: now also U5.3 (A2)
- net A7: now also U5.5 (E2)
- net GND: now also U4.2, U1.2 (GND), U5.8 (GND), U9.2 (GND)
- net nBE_DRV: now also U9.4, U9.6
- net nBE_IN: now also U7.6 (A4), U1.6 (IN2), U9.3
- net nBE_L: now also U9.1; no longer U7.6 (A4)
- net nIORQ: now also U5.4 (E1)
- net nM1: now also U5.6 (E3)
- net nMREQ: now also U1.3 (IN0); no longer U4.12
- net nMREQ_G: now also U1.4 (Y); no longer U4.11
- net nPRW: now also U4.3
- net nPW: now also U4.6
- net nRDROM: now also U4.11; no longer U4.6
- net PORT_A4 renamed PORT_SEL
- net PORT_SEL: now also U4.1, U4.4; no longer U4.10
- net nA4 renamed DEC_10
- net DEC_10: now also U5.14 (O1)
- new net DEC_00: JP4.1 (A), U5.15 (O0)
- no-connect marks 4 -> 8
Other:
- note added: "JP4: 1-2 (as shipped) answers $00-$0F, 2-3 answers $10-$1F. U8 C/D sections unused (inputs grounded)."
- note added: "The v2.2 bus logic (Logic.schdoc) rebuilt in 74LVC at 3.3 V: same logic at every Pico pin. /+W = I/O read of the card's port; /+RW = any I/O to it (not INTA)."
- note added: "U5 decodes the port (A7-A4, /IORQ, /M1); U4 makes /+RW, /+W, /RDROM; U1 /MREQ_G; U9 the open-drain /BE. U7 channel 5 = /BE_IN -> /BE_STAT."
- note removed: "JP4: 1-2 (as shipped) answers $00-$0F, 2-3 answers $10-$1F. U9B/U9C unused (inputs grounded). U8 C/D sections unused."
- note removed: "The v2.2 bus logic, gate for gate (Logic.schdoc). /+W = I/O read of the card's port; /+RW = any I/O to it; +X = port address match."
