File: hardware-v2.6/mcu.kicad_sch (KiCad schematic)
At the start: 45 parts, among them J1 USB-C, SW3 Pico Reset, SW4 BOOTSEL, U2 RP2040, U21 W25Q16JVSSIQ, U22 AMS1117-3.3, Y1 12MHz

Commit message: v2.6 prototype 2: glue logic in 74LVC, TPS3808 reset
The v2.2 glue (74LS04/27/32/09/157) is rebuilt in 74LVC at 3.3 V, because
the SN74LS09 (56) and XL74LS27 (108) were scarce at JLCPCB and every glue
output already ends at a 3.3 V part. Same logic at every Pico pin, so no
firmware change:

- U5 74LVC138 decodes the port (A4-A6 select; /IORQ, A7, /M1 enables);
  JP4 now picks output O0 ($00-$0F) or O1 ($10-$1F)
- U4 74LVC32: /+RW (buffered so it keeps step with /+W), /+W = /+RW-select
  OR /RD, /RDROM = A14 + A15 + /RD
- U1 74LVC1G97 (mux wired as OR with one inverted input): /MREQ_G
- U9 74LVC2G07 open-drain /BE driver; U7 channel 5 now carries /BE_IN as
  /BE_STAT, so R4 and R7 go
- U8 74LVC157 for the A14/A15 mux
- U11 TPS3808G01 replaces the 555, Q1 and passives: /RESET held below
  4.09 V and for 2.7 s after (CT 470 nF)

Checked by simulating the old and new netlists gate by gate over all
229,376 legal input states, both JP4 positions: all 12 outputs agree. The
only difference is /+W when /M1, /IORQ and /RD are all low, which a Z80
never does.

Layout: the RP2040's top/bottom-row IOVDD caps stand on their own pin's
lane with locked pin-to-cap stubs; without that the router left one net
open on three attempts. Routed first time, ERC/DRC clean at every
severity. 74 assembled parts (was 81), $9.79/board at 10.

Co-Authored-By: Claude Opus 5.5 <noreply@anthropic.com>
Parts:
- removed R4: 4k7, Resistor_SMD:R_0603_1608Metric, symbol Device:R
